File: garden-watering.kicad_sch (KiCad schematic)
At the start: 25 parts, among them J1 Barrel_Jack, J10 Conn_01x04, J11 Conn_01x05, J2 Conn_01x03, J7 Conn_01x04, J8 Conn_01x04, J9 Conn_01x04, U1 LM2576HVT-3.3, U2 ESP32-WROOM-32, U3 DHT11

Commit message: misc
Parts:
- removed C1: 100uF, Capacitor_THT:CP_Radial_D4.0mm_P2.00mm, symbol Device:C_Polarized
- removed C4: 1000uF, Capacitor_THT:CP_Radial_D4.0mm_P2.00mm, symbol Device:C_Polarized
- removed D1: MBR360, Diode_THT:D_DO-201AD_P12.70mm_Horizontal, symbol Device:D
- removed J1: Barrel_Jack, Connector_BarrelJack:BarrelJack_GCT_DCJ200-10-A_Horizontal, symbol Connector:Barrel_Jack
- removed L1: 330uH, Inductor_THT:L_Radial_D6.0mm_P4.00mm, symbol Device:L
- removed U1: LM2576HVT-3.3, Package_TO_SOT_THT:TO-220-5_Vertical, symbol Regulator_Switching:LM2576HVT-3.3
- added J7: JTAG, Connector_PinHeader_2.54mm:PinHeader_1x04_P2.54mm_Vertical, symbol Connector_Generic:Conn_01x04
- added R4 (x4): 100R, Resistor_THT:R_Axial_DIN0207_L6.3mm_D2.5mm_P7.62mm_Horizontal, symbol Device:R
- J1: renamed from J7; value Conn_01x04 -> GND
- J2: renamed from J10; value Conn_01x04 -> GND
- J3: renamed from J8; value Conn_01x04 -> +3.3V
- J4: renamed from J9; value Conn_01x04 -> +12V
- J5: renamed from J11; value Conn_01x05 -> GPIO
- J6: renamed from J2; value Conn_01x03 -> UART
- SW1: renamed from SW_RESET1; value SW_Push -> RESET
- SW2: renamed from SW_PROG1; value SW_Push -> PROG
- renumbered C5 to C1, C3 to C2, C2 to C3, U2 to U1, U3 to U2
Connections:
- net DHT: now also U1.29 (IO5); no longer U1.36 (IO22)
- net IO18: now also J5.1 (Pin_1); no longer J5.3 (Pin_3)
- net IO19: now also J5.2 (Pin_2); no longer J5.4 (Pin_4)
- net IO21: now also J5.3 (Pin_3); no longer J5.5 (Pin_5)
- net RELAY_1: now also U1.24 (IO2); no longer U1.27 (IO16)
- net RELAY_3: now also U1.27 (IO16); no longer U1.23 (IO15)
- net RELAY_4: now also U1.28 (IO17); no longer U1.24 (IO2)
- net MTMS: now reaches U1.13 (IO14)
- net MTMS: now also R4.1
- net MTDI: now reaches U1.14 (IO12)
- net MTDI: now also R4.1
- net MTCK: now reaches U1.16 (IO13)
- net MTCK: now also R4.1
- net IO23: now reaches U1.37 (IO23)
- net IO23: now also J5.5 (Pin_5)
- removed net IO17: J5.1 (Pin_1), U1.28 (IO17)
- removed net IO5: J5.2 (Pin_2), U1.29 (IO5)
- new net: J7.1 (Pin_1), R4.2
- new net: J7.4 (Pin_4), R4.2
- new net: J7.3 (Pin_3), R4.2
- new net: J7.2 (Pin_2), R4.2
- new net IO22: J5.4 (Pin_4), U1.36 (IO22)
- new net MTDO: R4.1, U1.23 (IO15)
- no-connect marks 19 -> 15
Other:
- added sheet Boost Converter (boost-converter.kicad_sch)
- added sheet USB-Power (usb-power.kicad_sch)
- moved on the sheet: C2, C3, J2, J3, J4
