File: relay.kicad_sch (KiCad schematic)
At the start: 10 parts, among them J3 Screw_Terminal_01x02, K1 SANYOU_SRD_Form_C, Q1 2N2222, SW1 SW_SPDT

Commit message: misc
Parts:
- renumbered D2 to D1, D3 to D2, D4 to D3, J3 to J8, R2 to R7, R3 to R8, R4 to R9, SW1 to SW3
