File: boost-converter.kicad_sch (KiCad schematic)
At the start: 5 parts, among them U4 LM2576T-12

Commit message: better footprint for hand soldering
Parts:
- U4: footprint Package_TO_SOT_THT:TO-220-5_Vertical -> Package_TO_SOT_THT:TO-220-5_P3.4x3.7mm_StaggerEven_Lead3.8mm_Vertical
Changed lines of the file:
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@@
       (effects (font (size 1.27 1.27)))
     )
-    (property "Footprint" "Package_TO_SOT_THT:TO-220-5_Vertical" (at 114.3 85.09 0)
+    (property "Footprint" "Package_TO_SOT_THT:TO-220-5_P3.4x3.7mm_StaggerEven_Lead3.8mm_Vertical" (at 114.3 85.09 0)
       (effects (font (size 1.27 1.27) italic) (justify left) hide)
     )
